Commit message: Add use_fake_hardware flag for backwards compatibility while adding new arg for hardware_type

File: urdf/robot/openarm_robot.xacro (robot description, xacro)
@@ -21,4 +21,5 @@
             ros2_control:=false
             can_interface:=''
+            hardware_type:='real'
             use_fake_hardware:=false
             fake_sensor_commands:=false
@@ -53,4 +54,7 @@
     <xacro:property name="arm_prefix_modified" value="${'' if arm_prefix == '' else arm_prefix + '_'}" />
     <xacro:property name="body_prefix_modified" value="${'' if body_prefix == '' else body_prefix + '_'}" />
+    <xacro:property
+        name="hardware"
+        value="${hardware_type if hardware_type != '' else ('mock' if use_fake_hardware else 'real')}" />
     <xacro:if value="${bimanual}">
         <xacro:openarm_body
@@ -100,5 +104,5 @@
             left_can_interface="${left_can_interface}"
             right_can_interface="${right_can_interface}"
-            use_fake_hardware="${use_fake_hardware}"
+            hardware_type="${hardware}"
             fake_sensor_commands="${fake_sensor_commands}"
             left_arm_prefix="${left_arm_prefix}"
@@ -154,5 +158,5 @@
             arm_prefix="${arm_prefix_modified}"
             can_interface="${can_interface}"
-            use_fake_hardware="${use_fake_hardware}"
+            hardware_type="${hardware}"
             fake_sensor_commands="${fake_sensor_commands}"
             hand="${hand}"
